Commit message: TODO: 轨迹规划时加入姿态

File: src/frcobot_description/urdf/fr5_robot.urdf (robot description, URDF)
Before this commit: robot fr5_robot, 8 links, 7 joints
Links:
- added link base_plate; collision box size=0.5 0.6 0.1; visual box size=0.5 0.6 0.1
- added link tool_Link
Joints:
- added joint base_to_plate: type fixed, parent base_link, child base_plate, origin xyz=0 0 -0.12 rpy=0 0 0
- added joint wrist3_to_tool: type fixed, parent wrist3_Link, child tool_Link, origin xyz=0 0 0.1 rpy=0 0 0
- joint j6: origin xyz=0 0 0.102 rpy=-1.570796 2.268928 0 -> xyz=0 0 0.102 rpy=-1.570796 0 0
